File: Ulticlone.brd (EAGLE design)
At the start: 100 x 80 mm, 104 parts, among them CON1 KLDX-0202-A-LT, IC1 ATMEGA2560-16AU, IC2 LM555D, J1 22-05-7028-02, J10 22-05-7028-02, J11 22-05-7028-02, J2 22-05-7028-02, J3 22-05-7028-02, J4 22-05-7028-02, J5 22-05-7028-02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

Commit message: updated
Parts:
- added R38, R39: 10k, rcl:R0603
- added SW1: (no value), SchlegelAr_Master:SW-SPDT-4MS1R202BM6NQNS
- R34, R36, R37: value 100 -> 1k
- R35: value 100 -> 10k
- moved C40 105.4 mm to (29.2, 72.4)
- moved C39 92.6 mm to (26.7, 64.8)
- moved C37 88.0 mm to (20.3, 71.1)
- moved C38 81.9 mm to (17.8, 62.2)
- moved CON1 80.0 mm to (12.7, 69.8)
- moved K1 75.7 mm to (41.4, 67.5), turned to 270 degrees
Connections:
- new net VCC/2: R38.1, SW1.1
- net ADC14: now also R38.2, R39.1
- net GND: now also R39.2
- net N$36: now also SW1.2
Changed lines of the file:
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@@
 <element name="Q3" library="transistor-npn" package="SOT23-BEC" value="BC817" x="93.98" y="41.91"/>
 <element name="R33" library="rcl" package="R0603" value="1k" x="96.52" y="41.91"/>
-<element name="K1" library="relay_finder_36_11" package="36.11" value="Finder 36.11.9.005.4011" x="90.66" y="10" rot="R90"/>
+<element name="K1" library="relay_finder_36_11" package="36.11" value="Finder 36.11.9.005.4011" x="41.42" y="67.47" rot="R270"/>
 <element name="D3" library="diode" package="SOD123" value="PMEG3010BER" x="80.01" y="5.08"/>
 <element name="Q4" library="transistor-pnp" package="SOT23-BEC" value="BC807-16SMD" x="78.74" y="11.43"/>
-<element name="R34" library="rcl" package="R0603" value="100" x="76.2" y="11.43"/>
-<element name="R35" library="rcl" package="R0603" value="100" x="68.58" y="13.97"/>
+<element name="R34" library="rcl" package="R0603" value="1k" x="76.2" y="11.43"/>
+<element name="R35" library="rcl" package="R0603" value="10k" x="68.58" y="13.97"/>
 <element name="IC2" library="linear" package="SO08" value="LM555D" x="71.12" y="10.16"/>
 <element name="C34" library="rcl" package="C0603K" value="100n" x="74.93" y="13.97"/>
 <element name="C35" library="rcl" package="C0603K" value="100n" x="67.31" y="10.16"/>
 <element name="C36" library="rcl" package="C0603K" value="100n" x="64.77" y="10.16"/>
-<element name="R36" library="rcl" package="R0603" value="100" x="62.23" y="10.16"/>
-<element name="R37" library="rcl" package="R0603" value="100" x="63.5" y="11.43"/>
+<element name="R36" library="rcl" package="R0603" value="1k" x="62.23" y="10.16"/>
+<element name="R37" library="rcl" package="R0603" value="1k" x="63.5" y="11.43"/>
 <element name="J10" library="con-molex" package="7395-02" value="22-05-7028-02" x="60.96" y="13.97">
 <attribute name="OC_NEWARK" value="unknown" x="60.96" y="13.97" size="1.778" layer="27" display="off"/>
@@
 <attribute name="OC_FARNELL" value="9731601" x="60.96" y="11.43" size="1.778" layer="27" display="off"/>
 </element>
-<element name="CON1" library="SchlegelAr_Master" package="KLDX-0202-A-LT" value="KLDX-0202-A-LT" x="11.43" y="-10.16"/>
-<element name="C37" library="SchlegelAr_Master" package="C_POL_4X4MM" value="100u/35V" x="-6.35" y="-12.7"/>
-<element name="C38" library="SchlegelAr_Master" package="C_POL_4X4MM" value="100u/35V" x="-15.24" y="-12.7"/>
-<element name="C39" library="SchlegelAr_Master" package="C_POL_4X4MM" value="10u" x="-24.13" y="-12.7"/>
-<element name="C40" library="SchlegelAr_Master" package="C_POL_4X4MM" value="10u" x="-33.02" y="-12.7"/>
+<element name="CON1" library="SchlegelAr_Master" package="KLDX-0202-A-LT" value="KLDX-0202-A-LT" x="12.7" y="69.85"/>
+<element name="C37" library="SchlegelAr_Master" package="C_POL_4X4MM" value="100u/35V" x="20.32" y="71.12"/>
+<element name="C38" library="SchlegelAr_Master" package="C_POL_4X4MM" value="100u/35V" x="17.78" y="62.23"/>
+<element name="C39" library="SchlegelAr_Master" package="C_POL_4X4MM" value="10u" x="26.67" y="64.77"/>
+<element name="C40" library="SchlegelAr_Master" package="C_POL_4X4MM" value="10u" x="29.21" y="72.39"/>
+<element name="R38" library="rcl" package="R0603" value="10k" x="8.89" y="54.61"/>
+<element name="R39" library="rcl" package="R0603" value="10k" x="11.43" y="58.42"/>
+<element name="SW1" library="SchlegelAr_Master" package="SW-SPDT-4MS1R202BM6NQNS" value="" x="7.62" y="58.42" rot="R270"/>
 </elements>
 <signals>
@@
 <contactref element="C39" pad="-"/>
 <contactref element="C40" pad="-"/>
+<contactref element="R39" pad="2"/>
 <wire x1="94.93" y1="31.92" x2="94.93" y2="40.81" width="0" layer="19" extent="1-1"/>
 <wire x1="84.695" y1="35.56" x2="94.93" y2="31.92" width="0" layer="19" extent="1-1"/>
@@
 <wire x1="18.655" y1="43.18" x2="16.115" y2="41.91" width="0" layer="19" extent="1-1"/>
 <wire x1="13.97" y1="27.94" x2="19.94" y2="34.02" width="0" layer="19" extent="1-1"/>
-<wire x1="96.66" y1="4.9" x2="81.91" y2="5.08" width="0" layer="19" extent="1-1"/>
-<wire x1="8.43" y1="-10.17" x2="13.97" y2="27.94" width="0" layer="19" extent="1-1"/>
-<wire x1="11.43" y1="-14.97" x2="8.43" y2="-10.17" width="0" layer="19" extent="1-1"/>
-<wire x1="-8.15" y1="-12.7" x2="8.43" y2="-10.17" width="0" layer="19" extent="1-1"/>
-<wire x1="-17.04" y1="-12.7" x2="-8.15" y2="-12.7" width="0" layer="19" extent="1-1"/>
-<wire x1="-25.93" y1="-12.7" x2="-17.04" y2="-12.7" width="0" layer="19" extent="1-1"/>
-<wire x1="-34.82" y1="-12.7" x2="-25.93" y2="-12.7" width="0" layer="19" extent="1-1"/>
+<wire x1="15.98" y1="62.23" x2="12.305" y2="48.26" width="0" layer="19" extent="1-1"/>
+<wire x1="12.7" y1="65.04" x2="15.98" y2="62.23" width="0" layer="19" extent="1-1"/>
+<wire x1="9.7" y1="69.84" x2="12.7" y2="65.04" width="0" layer="19" extent="1-1"/>
+<wire x1="18.52" y1="71.12" x2="12.7" y2="65.04" width="0" layer="19" extent="1-1"/>
+<wire x1="27.41" y1="72.39" x2="18.52" y2="71.12" width="0" layer="19" extent="1-1"/>
+<wire x1="35.42" y1="72.57" x2="27.41" y2="72.39" width="0" layer="19" extent="1-1"/>
+<wire x1="24.87" y1="64.77" x2="27.41" y2="72.39" width="0" layer="19" extent="1-1"/>
+<wire x1="12.28" y1="58.42" x2="13.97" y2="27.94" width="0" layer="19" extent="1-1"/>
 </signal>
 <signal name="VDD">
@@
 <signal name="ADC14">
 <contactref element="IC1" pad="83"/>
+<contactref element="R38" pad="2"/>
+<contactref element="R39" pad="1"/>
+<wire x1="9.74" y1="54.61" x2="30.44" y2="41.02" width="0" layer="19" extent="1-1"/>
+<wire x1="10.58" y1="58.42" x2="9.74" y2="54.61" width="0" layer="19" extent="1-1"/>
 </signal>
 <signal name="ADC13">
@@
 <contactref element="D3" pad="C"/>
 <contactref element="Q4" pad="C"/>
+<wire x1="78.74" y1="12.53" x2="47.42" y2="72.57" width="0" layer="19" extent="1-1"/>
 <wire x1="78.11" y1="5.08" x2="78.74" y2="12.53" width="0" layer="19" extent="1-1"/>
-<wire x1="84.66" y1="4.9" x2="78.11" y2="5.08" width="0" layer="19" extent="1-1"/>
 </signal>
 <signal name="N$36">
@@
 <contactref element="C38" pad="+"/>
 <contactref element="C37" pad="+"/>
-<wire x1="14.53" y1="-10.17" x2="96.66" y2="17.1" width="0" layer="19" extent="1-1"/>
-<wire x1="-4.55" y1="-12.7" x2="14.53" y2="-10.17" width="0" layer="19" extent="1-1"/>
-<wire x1="-13.44" y1="-12.7" x2="-4.55" y2="-12.7" width="0" layer="19" extent="1-1"/>
-<wire x1="-22.33" y1="-12.7" x2="-13.44" y2="-12.7" width="0" layer="19" extent="1-1"/>
-<wire x1="-31.22" y1="-12.7" x2="-22.33" y2="-12.7" width="0" layer="19" extent="1-1"/>
+<contactref element="SW1" pad="2"/>
+<wire x1="28.47" y1="64.77" x2="31.01" y2="72.39" width="0" layer="19" extent="1-1"/>
+<wire x1="35.42" y1="60.37" x2="28.47" y2="64.77" width="0" layer="19" extent="1-1"/>
+<wire x1="22.12" y1="71.12" x2="31.01" y2="72.39" width="0" layer="19" extent="1-1"/>
+<wire x1="15.8" y1="69.84" x2="22.12" y2="71.12" width="0" layer="19" extent="1-1"/>
+<wire x1="19.58" y1="62.23" x2="15.8" y2="69.84" width="0" layer="19" extent="1-1"/>
+<wire x1="7.62" y1="58.42" x2="19.58" y2="62.23" width="0" layer="19" extent="1-1"/>
 </signal>
 <signal name="+24V">
@@
 <wire x1="59.69" y1="11.43" x2="62.23" y2="13.97" width="0" layer="19" extent="1-1"/>
 </signal>
+<signal name="VCC/2">
+<contactref element="R38" pad="1"/>
+<contactref element="SW1" pad="1"/>
+<wire x1="7.62" y1="55.88" x2="8.04" y2="54.61" width="0" layer="19" extent="1-1"/>
+</signal>
 </signals>

Commit message: updated
Parts:
- moved SW1 1.27 mm to (7.62, 59.7)
Changed lines of the file:
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@@
 <layers>
 <layer number="1" name="Top" color="4" fill="1" visible="yes" active="yes"/>
+<layer number="2" name="Route2" color="1" fill="3" visible="no" active="no"/>
+<layer number="3" name="Route3" color="4" fill="3" visible="no" active="no"/>
+<layer number="14" name="Route14" color="1" fill="6" visible="no" active="no"/>
+<layer number="15" name="Route15" color="4" fill="6" visible="no" active="no"/>
 <layer number="16" name="Bottom" color="1" fill="1" visible="yes" active="yes"/>
 <layer number="17" name="Pads" color="2" fill="1" visible="yes" active="yes"/>
@@
 <element name="R38" library="rcl" package="R0603" value="10k" x="8.89" y="54.61"/>
 <element name="R39" library="rcl" package="R0603" value="10k" x="11.43" y="58.42"/>
-<element name="SW1" library="SchlegelAr_Master" package="SW-SPDT-4MS1R202BM6NQNS" value="" x="7.62" y="58.42" rot="R270"/>
+<element name="SW1" library="SchlegelAr_Master" package="SW-SPDT-4MS1R202BM6NQNS" value="" x="7.62" y="59.69" rot="R270"/>
 </elements>
 <signals>
@@
 <wire x1="15.8" y1="69.84" x2="22.12" y2="71.12" width="0" layer="19" extent="1-1"/>
 <wire x1="19.58" y1="62.23" x2="15.8" y2="69.84" width="0" layer="19" extent="1-1"/>
-<wire x1="7.62" y1="58.42" x2="19.58" y2="62.23" width="0" layer="19" extent="1-1"/>
+<wire x1="7.62" y1="59.69" x2="19.58" y2="62.23" width="0" layer="19" extent="1-1"/>
 </signal>
 <signal name="+24V">
@@
 <contactref element="R38" pad="1"/>
 <contactref element="SW1" pad="1"/>
-<wire x1="7.62" y1="55.88" x2="8.04" y2="54.61" width="0" layer="19" extent="1-1"/>
+<wire x1="7.62" y1="57.15" x2="8.04" y2="54.61" width="0" layer="19" extent="1-1"/>
 </signal>
 </signals>
