File: Ulticlone.sch (EAGLE design)
At the start: 104 parts, among them CON1 KLDX-0202-A-LT, IC1 ATMEGA2560-16AU, IC2 LM555D, J1 22-05-7028-02, J10 22-05-7028-02, J11 22-05-7028-02, J2 22-05-7028-02, J3 22-05-7028-02, J4 22-05-7028-02, J5 22-05-7028-02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

Commit message: updated
Parts:
- added R38, R39: 10k, rcl:R-EU_R0603
- added SW1: (no value), SchlegelAr_Master:SW-SPDT-4MS1R202BM6NQNS
- R34, R36, R37: value 100 -> 1k
- R35: value 100 -> 10k
Connections:
- new net VCC/2: R38.1, SW1.1
- net ADC14: now also R38.2, R39.1
- net GND: now also R39.2
- net N$36: now also SW1.2
Changed lines of the file:
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@@
 <part name="Q4" library="transistor-pnp" deviceset="BC807*" device="SMD" technology="-16"/>
 <part name="GND41" library="supply1" deviceset="GND" device=""/>
-<part name="R34" library="rcl" deviceset="R-EU_" device="R0603" value="100"/>
-<part name="R35" library="rcl" deviceset="R-EU_" device="R0603" value="100"/>
+<part name="R34" library="rcl" deviceset="R-EU_" device="R0603" value="1k"/>
+<part name="R35" library="rcl" deviceset="R-EU_" device="R0603" value="10k"/>
 <part name="IC2" library="linear" deviceset="*555" device="D" technology="LM"/>
 <part name="C34" library="rcl" deviceset="C-EU" device="C0603K" value="100n"/>
 <part name="C35" library="rcl" deviceset="C-EU" device="C0603K" value="100n"/>
 <part name="C36" library="rcl" deviceset="C-EU" device="C0603K" value="100n"/>
-<part name="R36" library="rcl" deviceset="R-EU_" device="R0603" value="100"/>
-<part name="R37" library="rcl" deviceset="R-EU_" device="R0603" value="100"/>
+<part name="R36" library="rcl" deviceset="R-EU_" device="R0603" value="1k"/>
+<part name="R37" library="rcl" deviceset="R-EU_" device="R0603" value="1k"/>
 <part name="GND42" library="supply1" deviceset="GND" device=""/>
 <part name="GND43" library="supply1" deviceset="GND" device=""/>
@@
 <part name="GND49" library="supply1" deviceset="GND" device=""/>
 <part name="GND50" library="supply1" deviceset="GND" device=""/>
+<part name="R38" library="rcl" deviceset="R-EU_" device="R0603" value="10k"/>
+<part name="R39" library="rcl" deviceset="R-EU_" device="R0603" value="10k"/>
+<part name="GND51" library="supply1" deviceset="GND" device=""/>
+<part name="P+23" library="supply1" deviceset="VCC/2" device=""/>
+<part name="SW1" library="SchlegelAr_Master" deviceset="SW-SPDT-4MS1R202BM6NQNS" device=""/>
 </parts>
 <sheets>
@@
 <instance part="GND49" gate="1" x="464.82" y="-7.62"/>
 <instance part="GND50" gate="1" x="474.98" y="-7.62"/>
+<instance part="R38" gate="G$1" x="502.92" y="-2.54" rot="R270"/>
+<instance part="R39" gate="G$1" x="502.92" y="-17.78" rot="R270"/>
+<instance part="GND51" gate="1" x="502.92" y="-27.94"/>
+<instance part="P+23" gate="G$1" x="502.92" y="10.16"/>
+<instance part="SW1" gate="SW" x="487.68" y="7.62"/>
 </instances>
 <busses>
@@
 <wire x1="474.98" y1="-5.08" x2="474.98" y2="-2.54" width="0.1524" layer="91"/>
 </segment>
+<segment>
+<pinref part="R39" gate="G$1" pin="2"/>
+<wire x1="502.92" y1="-22.86" x2="502.92" y2="-25.4" width="0.1524" layer="91"/>
+<pinref part="GND51" gate="1" pin="GND"/>
+</segment>
 </net>
 <net name="SCL" class="0">
@@
 <label x="101.6" y="149.86" size="1.27" layer="95" rot="R180" xref="yes"/>
 <pinref part="IC1" gate="1" pin="PK6(ADC14/PCINT22)"/>
+</segment>
+<segment>
+<pinref part="R38" gate="G$1" pin="2"/>
+<pinref part="R39" gate="G$1" pin="1"/>
+<wire x1="502.92" y1="-7.62" x2="502.92" y2="-10.16" width="0.1524" layer="91"/>
+<wire x1="502.92" y1="-10.16" x2="502.92" y2="-12.7" width="0.1524" layer="91"/>
+<wire x1="502.92" y1="-10.16" x2="505.46" y2="-10.16" width="0.1524" layer="91"/>
+<junction x="502.92" y="-10.16"/>
+<label x="505.46" y="-10.16" size="1.4224" layer="95" xref="yes"/>
 </segment>
 </net>
@@
 <wire x1="444.5" y1="5.08" x2="444.5" y2="7.62" width="0.1524" layer="91"/>
 <junction x="444.5" y="7.62"/>
+<pinref part="SW1" gate="SW" pin="2"/>
 </segment>
 </net>
@@
 </segment>
 </net>
+<net name="VCC/2" class="0">
+<segment>
+<pinref part="R38" gate="G$1" pin="1"/>
+<wire x1="502.92" y1="2.54" x2="502.92" y2="5.08" width="0.1524" layer="91"/>
+<pinref part="P+23" gate="G$1" pin="VCC/2"/>
+<pinref part="SW1" gate="SW" pin="1"/>
+<wire x1="502.92" y1="5.08" x2="502.92" y2="7.62" width="0.1524" layer="91"/>
+<wire x1="492.76" y1="5.08" x2="502.92" y2="5.08" width="0.1524" layer="91"/>
+<junction x="502.92" y="5.08"/>
+</segment>
+</net>
